File: bed_face-plate.sch (KiCad schematic (older format))
At the start: 52 parts

Commit message: initial plate from keebio dxf
Parts:
- removed H1, H2, H3, H4, H5: Hole, bed-face-components:screw_hole, symbol keebio:Hole
- removed MX1: ESC, bed-face-components:MX-1U-PlateCutout-EDIT, symbol MX_Alps_Hybrid:MX-NoLED
- removed MX10: O, bed-face-components:MX-1U-PlateCutout-EDIT, symbol MX_Alps_Hybrid:MX-NoLED
- removed MX11: P, bed-face-components:MX-1U-PlateCutout-EDIT, symbol MX_Alps_Hybrid:MX-NoLED
- removed MX12: BACKSPACE, bed-face-components:MX-1U-PlateCutout-EDIT, symbol MX_Alps_Hybrid:MX-NoLED
- removed MX13: TAB, bed-face-components:MX-1U-PlateCutout-EDIT, symbol MX_Alps_Hybrid:MX-NoLED
- removed MX14: A, bed-face-components:MX-1U-PlateCutout-EDIT, symbol MX_Alps_Hybrid:MX-NoLED
- removed MX15: S, bed-face-components:MX-1U-PlateCutout-EDIT, symbol MX_Alps_Hybrid:MX-NoLED
- removed MX16: D, bed-face-components:MX-1U-PlateCutout-EDIT, symbol MX_Alps_Hybrid:MX-NoLED
- removed MX17: F, bed-face-components:MX-1U-PlateCutout-EDIT, symbol MX_Alps_Hybrid:MX-NoLED
- removed MX18: G, bed-face-components:MX-1U-PlateCutout-EDIT, symbol MX_Alps_Hybrid:MX-NoLED
- removed MX19: H, bed-face-components:MX-1U-PlateCutout-EDIT, symbol MX_Alps_Hybrid:MX-NoLED
- removed MX2: Q, bed-face-components:MX-1U-PlateCutout-EDIT, symbol MX_Alps_Hybrid:MX-NoLED
- removed MX20: J, bed-face-components:MX-1U-PlateCutout-EDIT, symbol MX_Alps_Hybrid:MX-NoLED
- removed MX21: K, bed-face-components:MX-1U-PlateCutout-EDIT, symbol MX_Alps_Hybrid:MX-NoLED
- removed MX22: L, bed-face-components:MX-1U-PlateCutout-EDIT, symbol MX_Alps_Hybrid:MX-NoLED
- removed MX23: ; :, bed-face-components:MX-1U-PlateCutout-EDIT, symbol MX_Alps_Hybrid:MX-NoLED
- removed MX24: ' \", bed-face-components:MX-1U-PlateCutout-EDIT, symbol MX_Alps_Hybrid:MX-NoLED
- removed MX25: SHIFT, bed-face-components:MX-1U-PlateCutout-EDIT, symbol MX_Alps_Hybrid:MX-LED
- removed MX26: Z, bed-face-components:MX-1U-PlateCutout-EDIT, symbol MX_Alps_Hybrid:MX-NoLED
- removed MX27: X, bed-face-components:MX-1U-PlateCutout-EDIT, symbol MX_Alps_Hybrid:MX-NoLED
- removed MX28: C, bed-face-components:MX-1U-PlateCutout-EDIT, symbol MX_Alps_Hybrid:MX-NoLED
- removed MX29: V, bed-face-components:MX-1U-PlateCutout-EDIT, symbol MX_Alps_Hybrid:MX-NoLED
- removed MX3: W, bed-face-components:MX-1U-PlateCutout-EDIT, symbol MX_Alps_Hybrid:MX-NoLED
- removed MX30: B, bed-face-components:MX-1U-PlateCutout-EDIT, symbol MX_Alps_Hybrid:MX-NoLED
- removed MX31: N, bed-face-components:MX-1U-PlateCutout-EDIT, symbol MX_Alps_Hybrid:MX-NoLED
- removed MX32: M, bed-face-components:MX-1U-PlateCutout-EDIT, symbol MX_Alps_Hybrid:MX-NoLED
- removed MX33: , <, bed-face-components:MX-1U-PlateCutout-EDIT, symbol MX_Alps_Hybrid:MX-NoLED
- removed MX34: . >, bed-face-components:MX-1U-PlateCutout-EDIT, symbol MX_Alps_Hybrid:MX-NoLED
- removed MX35: / ?, bed-face-components:MX-1U-PlateCutout-EDIT, symbol MX_Alps_Hybrid:MX-NoLED
- removed MX36: ENTER, bed-face-components:MX-1U-PlateCutout-EDIT, symbol MX_Alps_Hybrid:MX-NoLED
- removed MX37: CTRL, bed-face-components:MX-1U-PlateCutout-EDIT, symbol MX_Alps_Hybrid:MX-NoLED
- removed MX38: GUI, bed-face-components:MX-1U-PlateCutout-EDIT, symbol MX_Alps_Hybrid:MX-NoLED
- removed MX39: ALT, bed-face-components:MX-1U-PlateCutout-EDIT, symbol MX_Alps_Hybrid:MX-NoLED
- removed MX4: E, bed-face-components:MX-1U-PlateCutout-EDIT, symbol MX_Alps_Hybrid:MX-NoLED
- removed MX40: FN, bed-face-components:MX-1U-PlateCutout-EDIT, symbol MX_Alps_Hybrid:MX-NoLED
- removed MX41: LOWER, bed-face-components:MX-1U-PlateCutout-EDIT, symbol MX_Alps_Hybrid:MX-NoLED
- removed MX42: SPACE, bed-face-components:MX-2U-PlateCutout-EDIT, symbol MX_Alps_Hybrid:MX-NoLED
- removed MX44: RAISE, bed-face-components:MX-1U-PlateCutout-EDIT, symbol MX_Alps_Hybrid:MX-NoLED
- removed MX45: LEFT, bed-face-components:MX-1U-PlateCutout-EDIT, symbol MX_Alps_Hybrid:MX-NoLED
- removed MX46: DOWN, bed-face-components:MX-1U-PlateCutout-EDIT, symbol MX_Alps_Hybrid:MX-NoLED
- removed MX47: UP, bed-face-components:MX-1U-PlateCutout-EDIT, symbol MX_Alps_Hybrid:MX-NoLED
- removed MX48: RIGHT, bed-face-components:MX-1U-PlateCutout-EDIT, symbol MX_Alps_Hybrid:MX-NoLED
- removed MX5: R, bed-face-components:MX-1U-PlateCutout-EDIT, symbol MX_Alps_Hybrid:MX-NoLED
- removed MX6: T, bed-face-components:MX-1U-PlateCutout-EDIT, symbol MX_Alps_Hybrid:MX-NoLED
- removed MX7: Y, bed-face-components:MX-1U-PlateCutout-EDIT, symbol MX_Alps_Hybrid:MX-NoLED
- removed MX8: U, bed-face-components:MX-1U-PlateCutout-EDIT, symbol MX_Alps_Hybrid:MX-NoLED
- removed MX9: I, bed-face-components:MX-1U-PlateCutout-EDIT, symbol MX_Alps_Hybrid:MX-NoLED
- added H1, H2, H3, H4, H5: MountingHole_Pad, bed-face-components:2.1mm_Screw_Hole, symbol Mechanical:MountingHole_Pad
- added P1: plate, bed-face-components:plate, symbol bed_face_plate:plate
Connections:
- new net GND: H1.1, H2.1, H3.1, H4.1, H5.1
